File: weird65.kicad_pcb (KiCad board)
At the start: 2 copper layers, 246.8 x 112.4 mm, 72 parts, among them SW1 SW_Diode, SW10 SW_Diode, SW11 SW_Diode, SW12 SW_Diode, SW13 SW_Diode, SW14 SW_Diode, SW15 SW_Diode, SW16 SW_Diode, SW17 SW_Diode, SW18 SW_Diode, SW19 SW_Diode, SW2 SW_Diode, SW20 SW_Diode, SW21 SW_Diode, SW22 SW_Diode, SW23 SW_Diode, SW24 SW_Diode, SW25 SW_Diode, SW27 SW_Diode, SW28 SW_Diode, SW29 SW_Diode, SW3 SW_Diode, SW30 SW_Diode, SW31 SW_Diode, SW32 SW_Diode, SW33 SW_Diode, SW34 SW_Diode, SW35 SW_Diode, SW36 SW_Diode, SW37 SW_Diode, SW38 SW_Diode, SW39 SW_Diode, SW4 SW_Diode, SW40 SW_Diode, SW41 SW_Diode, SW42 SW_Diode, SW43 SW_Diode, SW44 SW_Diode, SW45 SW_Diode, SW46 SW_Diode, SW47 SW_Diode, SW48 SW_Diode, SW49 SW_Diode, SW5 SW_Diode, SW53 SW_Diode, SW54 SW_Diode, SW55 SW_Diode, SW56 SW_Diode, SW57 SW_Diode, SW59 SW_Diode, SW6 SW_Diode, SW61 SW_Diode, SW62 SW_Diode, SW63 SW_Diode, SW65 SW_Diode, SW67 SW_Diode, SW68 SW_Diode, SW69 SW_Diode, SW7 SW_Diode, SW71 SW_Diode, SW72 SW_Diode, SW73 SW_Diode, SW74 SW_Diode, SW8 SW_Diode, SW9 SW_Diode

Commit message: moved the promicro to the left
Parts:
- moved MCU1 114.8 mm to (465.7, 288.4)
Changed lines of the file:
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@@
   )
   (footprint "customs:ProMicro" (layer "F.Cu")
-    (at 580.5 288.392 -90)
+    (at 465.74 288.392 -90)
     (attr through_hole)
     (fp_text reference "MCU1" (at 0 0 90) (layer "F.SilkS") hide
